File: Pathfinder.kicad_sch (KiCad schematic)
At the start: 0 parts

Commit message: Add files via upload
Parts:
- added D1, D2, D3: L08R5000Q1, L08R5000Q1:LEDRD254W57D500H1070, symbol L08R5000Q1:L08R5000Q1
- added R1, R2, R3: R, symbol Device:R
- added SW1: SW_Push, symbol Switch:SW_Push
- added U1: XIAO-RP2040-DIP, Module:MOUDLE14P-XIAO-DIP-SMD, symbol Seeed_Studio_XIAO_Series:XIAO-RP2040-DIP
Connections:
- new net: R1.1, SW1.1
- new net: D2.A, R2.1
- new net: D3.A, R3.1
