File: Pathfinder.kicad_pcb (KiCad board)
At the start: 2 copper layers, 0 parts

Commit message: Add files via upload
Parts:
- added D1: L08R5000Q1, footprints:LEDRD254W57D500H1070, F.Cu at (109.5, 70.5)
- added D2: L08R5000Q1, footprints:LEDRD254W57D500H1070, F.Cu at (134.2, 72.0)
- added D3: L08R5000Q1, footprints:LEDRD254W57D500H1070, F.Cu at (153.7, 72.0)
- added R1: R, Resistor_THT:R_Axial_DIN0204_L3.6mm_D1.6mm_P5.08mm_Horizontal, F.Cu at (108.0, 103.5)
- added R2: R, Resistor_THT:R_Axial_DIN0204_L3.6mm_D1.6mm_P5.08mm_Horizontal, F.Cu at (132.0, 103.0)
- added R3: R, Resistor_THT:R_Axial_DIN0204_L3.6mm_D1.6mm_P5.08mm_Horizontal, F.Cu at (156.5, 103.0)
- added SW1: SW_Push, Button_Switch_Keyboard:SW_Cherry_MX_1.00u_PCB, F.Cu at (113.0, 84.5)
- added SW2: SW_Push, Button_Switch_Keyboard:SW_Cherry_MX_1.00u_PCB, F.Cu at (137.0, 84.5)
- added SW3: SW_Push, Button_Switch_Keyboard:SW_Cherry_MX_1.00u_PCB, F.Cu at (161.3, 84.5)
- added U1: XIAO-RP2040-DIP, footprints:XIAO-RP2040-DIP, F.Cu at (134.4, 56.1)
Routing:
- net LED2: track 0.00 -> 213.3 mm
- net LED1: track 0.00 -> 172.6 mm
- net button3: track 0.00 -> 82.9 mm
- net button2: track 0.00 -> 61.2 mm
- net button1: track 0.00 -> 42.3 mm
- net LED3: track 0.00 -> 1.08 mm
