File: Pathfinder.kicad_pcb (KiCad board)
At the start: 2 copper layers, 10 parts, among them SW1 SW_Push, SW2 SW_Push, SW3 SW_Push, U1 XIAO-RP2040-DIP

Commit message: Add files via upload
Parts:
- moved R1 26.0 mm to (107.5, 77.5)
- moved R2 25.5 mm to (131.9, 77.5)
- moved R3 25.5 mm to (156.4, 77.5)
- moved D3 5.02 mm to (158.7, 71.5)
- moved D1 1.52 mm to (109.8, 72.0)
Routing:
- net LED2: track 213.3 -> 23.9 mm, vias 0 -> 1
- net LED1: track 172.6 -> 27.3 mm
- net GND: track 0.11 -> 141.4 mm
- net LED3: track 1.08 -> 43.4 mm, vias 0 -> 1
- net button3: track 82.9 -> 47.4 mm, vias 0 -> 1
- net button2: track 61.2 -> 41.8 mm
- net Net-(D3-PadA): track 0.00 -> 7.48 mm
- net Net-(D2-PadA): track 0.00 -> 6.98 mm
- net Net-(D1-PadA): track 0.00 -> 6.98 mm
- net button1: track 42.3 -> 46.8 mm
